File: ee372b-ldo-testbench/ee372b-ldo-testbench.kicad_pcb (KiCad board)
At the start: 4 copper layers, 136 parts, among them J1 PEC02SAAN, J10 OUT_S, J11 VOUT, J12 VDD_BUF, J13 V_SIG, J14 PEC03SAAN, J15 VSIG_BUF, J16 PEC03SAAN, J17 PEC03SAAN, J18 PEC03SAAN, J19 PEC03SAAN, J2 PEC02SAAN, J20 VREF_EXTERNAL, J21 PEC02SAAN, J22 PEC02SAAN, J23 PEC02SAAN, J24 PEC02SAAN, J25 PEC03SAAN, J3 GND, J4 1V8, J5 3v3_EXTERNAL, J8 VIN, J9 IN_S, Q1 FDV305N, Q2 FDV305N, Q3 FDV305N, Q4 FDV305N, Q5 FDV305N, U1 MMSZ4679T1G, U3 ADS1220IPW, U4 BUF634AIDR

Commit message: reduced pin bypass caps
Parts:
- removed C24, C9: 100nF, Capacitor_SMD:C_0805_2012Metric_Pad1.18x1.45mm_HandSolder
- removed R21, R22, R23, R24, R25, R26, R27, R28, R29, R30, R31, R32, R33, R34, R35, R36: 0, Resistor_SMD:R_0805_2012Metric_Pad1.20x1.40mm_HandSolder
- added R45: 0, Resistor_SMD:R_0805_2012Metric_Pad1.20x1.40mm_HandSolder, F.Cu at (521.5, 98.5)
- added R46: 0, Resistor_SMD:R_0805_2012Metric_Pad1.20x1.40mm_HandSolder, F.Cu at (526.5, 99.0)
- C27: value 1uF -> 100nF
- C6: value 100nF -> 1uF
- moved C27 78.8 mm to (544.0, 88.5), turned to -90 degrees
- moved C23 78.0 mm to (547.5, 88.5), turned to 90 degrees
- moved C17 68.8 mm to (552.5, 93.5), turned to 180 degrees
- moved C5 66.7 mm to (540.5, 96.0)
- moved C6 66.0 mm to (540.9, 99.5)
- moved C7 64.9 mm to (548.0, 100.5), turned to 90 degrees
- moved C10 62.2 mm to (552.5, 97.5), turned to 180 degrees
- moved C4 3.00 mm to (540.5, 93.5)
Connections:
- C17 pad 2: Net-(C17-Pad2) -> Net-(C10-Pad2)
- C23 pad 2: Net-(C23-Pad2) -> Net-(C10-Pad2)
- C27 pad 2: Net-(C24-Pad2) -> Net-(C10-Pad2)
- C4 pad 2: /c1_vin_jump -> Net-(C10-Pad2)
- C5 pad 2: Net-(C5-Pad2) -> Net-(C10-Pad2)
- C6 pad 2: Net-(C6-Pad2) -> Net-(C10-Pad2)
- C7 pad 2: Net-(C7-Pad2) -> Net-(C10-Pad2)
- U2 pad 1: Net-(R21-Pad1) -> GND
- U2 pad 13: Net-(R26-Pad1) -> GND
- U2 pad 14: Net-(C6-Pad2) -> Net-(C10-Pad2)
- U2 pad 16: Net-(C7-Pad2) -> Net-(C10-Pad2)
- U2 pad 17: Net-(C9-Pad2) -> Net-(C10-Pad2)
- U2 pad 18: Net-(R27-Pad1) -> GND
- U2 pad 2: /c1_vin_jump -> Net-(C10-Pad2)
- U2 pad 20: Net-(R28-Pad1) -> GND
- U2 pad 22: Net-(R29-Pad1) -> GND
- U2 pad 23: Net-(R30-Pad1) -> GND
- U2 pad 24: Net-(C17-Pad2) -> Net-(C10-Pad2)
- U2 pad 25: Net-(R31-Pad1) -> GND
- U2 pad 26: Net-(R32-Pad1) -> GND
- U2 pad 27: Net-(C23-Pad2) -> Net-(C10-Pad2)
- U2 pad 28: Net-(R33-Pad1) -> GND
- U2 pad 29: Net-(R34-Pad1) -> GND
- U2 pad 3: Net-(R22-Pad1) -> GND
- U2 pad 30: Net-(R35-Pad1) -> GND
- U2 pad 31: Net-(R36-Pad1) -> GND
- U2 pad 32: Net-(C24-Pad2) -> Net-(C10-Pad2)
- U2 pad 4: Net-(R23-Pad1) -> GND
- U2 pad 6: Net-(R24-Pad1) -> GND
- U2 pad 7: Net-(R25-Pad1) -> GND
- U2 pad 8: Net-(C5-Pad2) -> Net-(C10-Pad2)
- U3 pad 6: GND -> /LDO_GND

Commit message: added 100mm x 100mm thing
Parts:
- removed J8: VIN, 1_EE372_DemoBoard:CALTEST_CT3151-2
- removed R57: 0, Resistor_SMD:R_0805_2012Metric_Pad1.20x1.40mm_HandSolder
- TP10: value 1V8 -> 3V3
- TP3: value OUT_S1 -> LOAD_OUT
- TP4: value OUT_S2 -> LDO_VOUT
- moved J12 597.3 mm to (471.9, 102.5)
- moved J3 393.4 mm to (471.9, 132.5), turned to -90 degrees
- moved J4 358.7 mm to (472.0, 87.5), turned to -90 degrees
- moved J5 309.1 mm to (471.9, 117.5), turned to -90 degrees
- moved TP10 305.7 mm to (485.5, 118.5)
- moved TP7 304.1 mm to (485.0, 84.5)
- moved TP6 302.8 mm to (485.0, 89.5)
- moved J11 243.6 mm to (563.1, 87.5), turned to 90 degrees
- moved R59 200.2 mm to (556.5, 80.0)
- moved TP4 198.6 mm to (549.0, 103.5)
- moved TP3 198.6 mm to (549.0, 98.5)
- moved J10 174.3 mm to (544.5, 78.0)
- moved C26 124.5 mm to (473.5, 81.0), turned to 180 degrees
- moved R51 98.9 mm to (514.0, 103.0), turned to 90 degrees
- moved J20 97.6 mm to (527.0, 116.0)
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Connections:
- net /VIN renamed /1V8
- R37 pad 2: Net-(U2-OTA_VREF) -> /BGR_VREF
- U2 pad 19: Net-(U2-OTA_VREF) -> /BGR_VREF

Commit message: Add files via upload
Parts:
- moved R56 424.0 mm to (14.6, 80.8)
- moved J9 409.1 mm to (32.7, 80.3)
- moved TP1 409.1 mm to (25.0, 78.3)
- moved TP2 409.1 mm to (25.0, 83.2)
- moved J12 392.4 mm to (84.2, 41.6), turned to 180 degrees
- moved C11 385.8 mm to (42.8, 101.5)
- moved U1 381.9 mm to (26.3, 91.8), turned to 0 degrees
- moved J20 348.5 mm to (182.5, 63.3)
- moved J4 341.0 mm to (136.1, 29.3)
- moved R37 331.7 mm to (193.9, 61.8)
- moved C10 331.7 mm to (200.5, 40.3)
- moved C17 331.7 mm to (200.5, 36.3)
- moved C23 331.7 mm to (195.5, 31.3)
- moved C26 331.7 mm to (146.0, 28.3)
- moved C27 331.7 mm to (192.0, 31.4)
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
Commit message: added selectable output for ADC Analog3 pin measurement for VOUT
Parts:
- moved H3 339.1 mm to (235.0, 22.0)
- moved H2 291.2 mm to (235.0, 112.0)
- moved H4 278.6 mm to (145.0, 22.0)
- moved H1 219.3 mm to (145.0, 112.0)
- moved R17 202.3 mm to (227.9, 79.2), turned to 0 degrees
- moved R15 196.3 mm to (227.9, 77.0), turned to 0 degrees
- moved R14 190.9 mm to (227.9, 75.0), turned to 0 degrees
- moved R12 185.3 mm to (227.9, 72.8), turned to 0 degrees
- moved R20 184.8 mm to (218.2, 79.4), turned to 0 degrees
- moved R10 179.9 mm to (227.9, 70.8), turned to 0 degrees
- moved R19 179.3 mm to (218.1, 77.2), turned to 0 degrees
- moved R18 174.4 mm to (218.2, 75.2), turned to 0 degrees
- moved R16 171.4 mm to (218.2, 73.0), turned to 0 degrees
- moved Q5 171.1 mm to (190.0, 68.8)
- moved J19 169.9 mm to (189.7, 79.9)
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Other:
- board text added: "to: EXT"
- board text added: "to: VIN"
