File: ee372b-ldo-testbench/ee372b-ldo-testbench.kicad_sch (KiCad schematic)
At the start: 128 parts, among them J1 PEC02SAAN, J10 OUT_S, J11 VOUT, J12 VDD_BUF, J13 V_SIG, J14 PEC03SAAN, J15 VSIG_BUF, J16 PEC03SAAN, J17 PEC03SAAN, J18 PEC03SAAN, J19 PEC03SAAN, J2 PEC02SAAN, J20 VREF_EXTERNAL, J21 PEC02SAAN, J22 PEC02SAAN, J23 PEC02SAAN, J24 PEC02SAAN, J25 PEC03SAAN, J3 GND, J4 1V8, J5 3v3_EXTERNAL, J6 GND, J9 IN_S, Q1 FDV305N, Q2 FDV305N, Q3 FDV305N, Q4 FDV305N, Q5 FDV305N, U1 MMSZ4679T1G, U3 ADS1220IPW, U4 BUF634AIDR

Commit message: final submitted
Parts:
- added TP18, TP19: TestPoint_Probe, TestPoint:TestPoint_Pad_D1.0mm, symbol Connector:TestPoint_Probe
Connections:
- net LDO_VOUT: now also TP18.1
- net VOUT: now also TP19.1
Changed lines of the file:
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@@
 	)
 	(junction
+		(at 515.62 110.49)
+		(diameter 0)
+		(color 0 0 0 0)
+	)
+	(junction
 		(at 46.99 312.42)
 		(diameter 0)
@@
 	)
 	(junction
+		(at 499.11 110.49)
+		(diameter 0)
+		(color 0 0 0 0)
+	)
+	(junction
 		(at 476.25 110.49)
 		(diameter 0)
@@
 	(wire
 		(pts
+			(xy 499.11 97.79) (xy 499.11 110.49)
+		)
+		(stroke
+			(width 0)
+			(type default)
+		)
+	)
+	(wire
+		(pts
 			(xy 354.33 80.01) (xy 354.33 83.82)
 		)
@@
 	(wire
 		(pts
+			(xy 499.11 110.49) (xy 500.38 110.49)
+		)
+		(stroke
+			(width 0)
+			(type default)
+		)
+	)
+	(wire
+		(pts
 			(xy 396.24 107.95) (xy 396.24 110.49)
 		)
@@
 	(wire
 		(pts
-			(xy 490.22 110.49) (xy 500.38 110.49)
+			(xy 490.22 110.49) (xy 499.11 110.49)
 		)
 		(stroke
@@
 	(wire
 		(pts
+			(xy 515.62 97.79) (xy 515.62 110.49)
+		)
+		(stroke
+			(width 0)
+			(type default)
+		)
+	)
+	(wire
+		(pts
 			(xy 78.74 312.42) (xy 78.74 314.96)
 		)
@@
 	(wire
 		(pts
+			(xy 515.62 110.49) (xy 520.7 110.49)
+		)
+		(stroke
+			(width 0)
+			(type default)
+		)
+	)
+	(wire
+		(pts
 			(xy 255.27 303.53) (xy 264.16 303.53)
 		)
@@
 	(wire
 		(pts
-			(xy 508 110.49) (xy 520.7 110.49)
+			(xy 508 110.49) (xy 515.62 110.49)
 		)
 		(stroke
@@
 	)
 	(symbol
+		(lib_id "Connector:TestPoint_Probe")
+		(at 515.62 97.79 0)
+		(unit 1)
+		(body_style 1)
+		(exclude_from_sim no)
+		(in_bom yes)
+		(on_board yes)
+		(in_pos_files yes)
+		(dnp no)
+		(fields_autoplaced yes)
+		(property "Reference" "TP19"
+			(at 519.43 94.9324 0)
+			(show_name no)
+			(do_not_autoplace no)
+			(effects
+				(font
+					(size 1.27 1.27)
+				)
+				(justify left)
+			)
+		)
+		(property "Value" "TestPoint_Probe"
+			(at 519.43 97.4724 0)
+			(show_name no)
+			(do_not_autoplace no)
+			(effects
+				(font
+					(size 1.27 1.27)
+				)
+				(justify left)
+			)
+		)
+		(property "Footprint" "TestPoint:TestPoint_Pad_D1.0mm"
+			(at 520.7 97.79 0)
+			(hide yes)
+			(show_name no)
+			(do_not_autoplace no)
+			(effects
+				(font
+					(size 1.27 1.27)
+				)
+			)
+		)
+		(property "Datasheet" ""
+			(at 520.7 97.79 0)
+			(hide yes)
+			(show_name no)
+			(do_not_autoplace no)
+			(effects
+				(font
+					(size 1.27 1.27)
+				)
+			)
+		)
+		(property "Description" "test point (alternative probe-style design)"
+			(at 515.62 97.79 0)
+			(hide yes)
+			(show_name no)
+			(do_not_autoplace no)
+			(effects
+				(font
+					(size 1.27 1.27)
+				)
+			)
+		)
+		(pin "1"
+		)
+		(instances
+			(project "ee372b-ldo-testbench"
+				(path "/4eaac8a8-2761-424f-b17c-d4cc8c253812"
+					(reference "TP19")
+					(unit 1)
+				)
+			)
+		)
+	)
+	(symbol
 		(lib_id "Device:C_Small_US")
 		(at 356.87 71.12 0)
@@
 					(unit 1)
 				)
+			)
+		)
+	)
+	(symbol
+		(lib_id "Connector:TestPoint_Probe")
+		(at 499.11 97.79 0)
+		(unit 1)
+		(body_style 1)
+		(exclude_from_sim no)
+		(in_bom yes)
+		(on_board yes)
+		(in_pos_files yes)
+		(dnp no)
+		(fields_autoplaced yes)
+		(property "Reference" "TP18"
+			(at 502.92 94.9324 0)
+			(show_name no)
+			(do_not_autoplace no)
+			(effects
+				(font
+					(size 1.27 1.27)
+				)
+				(justify left)
+			)
+		)
+		(property "Value" "TestPoint_Probe"
+			(at 502.92 97.4724 0)
+			(show_name no)
+			(do_not_autoplace no)
+			(effects
+				(font
+					(size 1.27 1.27)
+				)
+				(justify left)
+			)
+		)
+		(property "Footprint" "TestPoint:TestPoint_Pad_D1.0mm"
+			(at 504.19 97.79 0)
+			(hide yes)
+			(show_name no)
+			(do_not_autoplace no)
+			(effects
+				(font
+					(size 1.27 1.27)
+				)
+			)
+		)
+		(property "Datasheet" ""
+			(at 504.19 97.79 0)
+			(hide yes)
+			(show_name no)
+			(do_not_autoplace no)
+			(effects
+				(font
+					(size 1.27 1.27)
+				)
+			)
+		)
+		(property "Description" "test point (alternative probe-style design)"
+			(at 499.11 97.79 0)
+			(hide yes)
+			(show_name no)
+			(do_not_autoplace no)
+			(effects
+				(font
+					(size 1.27 1.27)
+				)
+			)
+		)
+		(pin "1"
+		)
+		(instances
+			(project "ee372b-ldo-testbench"
+				(path "/4eaac8a8-2761-424f-b17c-d4cc8c253812"
+					(reference "TP18")
+					(unit 1)
+				)
