File: ee372b-ldo-testbench/_restore_backup_2026-10-05T01-44-18-442/ee372b-ldo-testbench.kicad_sch (KiCad schematic)
At the start: 128 parts, among them J1 PEC02SAAN, J10 OUT_S, J11 VOUT, J12 VDD_BUF, J13 V_SIG, J14 PEC03SAAN, J15 VSIG_BUF, J16 PEC03SAAN, J17 PEC03SAAN, J18 PEC03SAAN, J19 PEC03SAAN, J2 PEC02SAAN, J20 VREF_EXTERNAL, J21 PEC02SAAN, J22 PEC02SAAN, J23 PEC02SAAN, J24 PEC02SAAN, J25 PEC03SAAN, J3 GND, J4 1V8, J5 3v3_EXTERNAL, J6 GND, J9 IN_S, Q1 FDV305N, Q2 FDV305N, Q3 FDV305N, Q4 FDV305N, Q5 FDV305N, U1 MMSZ4679T1G, U3 ADS1220IPW, U4 BUF634AIDR

Commit message: omg cleared DRC
Connections:
- net GND: no longer A1.13 (GND), A1.18 (GND), A1.23 (GND), A1.28 (GND), A1.3 (GND), A1.38 (GND), A1.8 (GND), C3.1
- new net: A1.13 (GND), A1.18 (GND), A1.23 (GND), A1.28 (GND), A1.3 (GND), A1.38 (GND), A1.8 (GND), C3.1
Other:
- moved on the sheet: C3
Changed lines of the file:
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@@
 	)
 	(junction
-		(at 236.22 342.9)
-		(diameter 0)
-		(color 0 0 0 0)
-	)
-	(junction
 		(at 215.9 182.88)
 		(diameter 0)
@@
 	(wire
 		(pts
-			(xy 236.22 342.9) (xy 232.41 341.63)
-		)
-		(stroke
-			(width 0)
-			(type default)
-		)
-	)
-	(wire
-		(pts
 			(xy 132.08 290.83) (xy 132.08 292.1)
 		)
@@
 	(wire
 		(pts
-			(xy 236.22 350.52) (xy 232.41 350.52)
-		)
-		(stroke
-			(width 0)
-			(type default)
-		)
-	)
-	(wire
-		(pts
 			(xy 229.87 76.2) (xy 229.87 80.01)
 		)
@@
 	(wire
 		(pts
-			(xy 219.71 342.9) (xy 236.22 342.9)
-		)
-		(stroke
-			(width 0)
-			(type default)
-		)
-	)
-	(wire
-		(pts
 			(xy 82.55 114.3) (xy 86.36 114.3)
 		)
@@
 	(wire
 		(pts
+			(xy 232.41 349.25) (xy 232.41 354.33)
+		)
+		(stroke
+			(width 0)
+			(type default)
+		)
+	)
+	(wire
+		(pts
 			(xy 533.4 110.49) (xy 548.64 110.49)
 		)
@@
 	(wire
 		(pts
-			(xy 232.41 350.52) (xy 232.41 364.49)
-		)
-		(stroke
-			(width 0)
-			(type default)
-		)
-	)
-	(wire
-		(pts
 			(xy 335.28 67.31) (xy 341.63 67.31)
 		)
@@
 	)
 	(label "3V3_PICO"
-		(at 232.41 364.49 90)
+		(at 232.41 354.33 90)
 		(effects
 			(font
@@
 		)
 	)
-	(label "GND"
-		(at 219.71 342.9 180)
-		(effects
-			(font
-				(size 1.27 1.27)
-			)
-			(justify right bottom)
-		)
-	)
 	(label "VG4"
 		(at 124.46 299.72 0)
@@
 	(symbol
 		(lib_id "Device:C")
-		(at 236.22 346.71 0)
+		(at 232.41 345.44 0)
 		(unit 1)
 		(body_style 1)
@@
 		(fields_autoplaced yes)
 		(property "Reference" "C3"
-			(at 240.03 345.4399 0)
+			(at 236.22 344.1699 0)
 			(show_name no)
 			(do_not_autoplace no)
@@
 		)
 		(property "Value" "0.1uF"
-			(at 240.03 347.9799 0)
+			(at 236.22 346.7099 0)
 			(show_name no)
 			(do_not_autoplace no)
@@
 		)
 		(property "Footprint" "Capacitor_SMD:C_0805_2012Metric_Pad1.18x1.45mm_HandSolder"
-			(at 237.1852 350.52 0)
+			(at 233.3752 349.25 0)
 			(hide yes)
 			(show_name no)
@@
 		)
 		(property "Datasheet" ""
-			(at 236.22 346.71 0)
+			(at 232.41 345.44 0)
 			(hide yes)
 			(show_name no)
@@
 		)
 		(property "Description" "Unpolarized capacitor"
-			(at 236.22 346.71 0)
+			(at 232.41 345.44 0)
 			(hide yes)
 			(show_name no)
@@
 		(in_pos_files yes)
 		(dnp no)
+		(fields_autoplaced yes)
 		(property "Reference" "C21"
 			(at 97.79 86.3599 0)
@@
 		)
 		(property "Value" "100nF"
-			(at 86.36 87.884 0)
+			(at 97.79 88.8999 0)
 			(show_name no)
 			(do_not_autoplace no)
